Commit message: cleaned up packages for presentation

File: simbot_description/src/description/simbot_description.urdf (robot description, URDF)
Before this commit: robot simbot, 10 links, 9 joints
Links:
- removed link cam_rgb_frame
- removed link cam_rgb_link
- removed link cam_rgb_optical_frame
Joints:
- removed joint cam_rgb_base_link_joint
- removed joint cam_rgb_joint
- removed joint cam_rgb_optical_joint
